Commit message: Worked on ar mvisualization some more

File: src/pick_up/urdf/Hiwonder.urdf (robot description, URDF)
Before this commit: robot xarm, 6 links, 5 joints
Links:
- link xarm_2_link: geometry collision cylinder length=0.05 radius=0.01; visual cylinder length=0.05 radius=0.01
- link xarm_3_link: geometry collision cylinder length=0.05 radius=0.01; visual cylinder length=0.05 radius=0.01
- link xarm_4_link: geometry collision cylinder length=0.05 radius=0.01; visual cylinder length=0.05 radius=0.01
- link xarm_5_link: geometry collision cylinder length=0.05 radius=0.01; visual cylinder length=0.05 radius=0.01
- link xarm_6_link: geometry collision cylinder length=0.05 radius=0.01; visual cylinder length=0.05 radius=0.01
- link xarm_base_link: geometry collision cylinder length=0.05 radius=0.01; visual cylinder length=0.05 radius=0.01
