Commit message: Added proper simulation

File: src/pick_up/urdf/Arm.urdf (robot description, URDF)
Before this commit: robot armpi_fpv, 15 links, 14 joints
Links:
- link base_link: geometry collision mesh filename=package://pick_up/meshes/base_link.STL; visual mesh filename=package://pick_up/meshes/base_link.STL
- link camera_link: geometry collision mesh filename=package://pick_up/meshes/camera_link.STL; visual mesh filename=package://pick_up/meshes/camera_link.STL
- link gripper_base: geometry collision mesh filename=package://pick_up/meshes/gripper_base.STL; visual mesh filename=package://pick_up/meshes/gripper_base.STL
- link l_in_link: geometry collision mesh filename=package://pick_up/meshes/l_in_link.STL; visual mesh filename=package://pick_up/meshes/l_in_link.STL
- link l_link: geometry collision mesh filename=package://pick_up/meshes/l_link.STL; visual mesh filename=package://pick_up/meshes/l_link.STL
- link l_out_link: geometry collision mesh filename=package://pick_up/meshes/l_out_link.STL; visual mesh filename=package://pick_up/meshes/l_out_link.STL
- link link1: geometry collision mesh filename=package://pick_up/meshes/link1.STL; visual mesh filename=package://pick_up/meshes/link1.STL
- link link2: geometry collision mesh filename=package://pick_up/meshes/link2.STL; visual mesh filename=package://pick_up/meshes/link2.STL
- link link3: geometry collision mesh filename=package://pick_up/meshes/link3.STL; visual mesh filename=package://pick_up/meshes/link3.STL
- link link4: geometry collision mesh filename=package://pick_up/meshes/link4.STL; visual mesh filename=package://pick_up/meshes/link4.STL
- link link5: geometry collision mesh filename=package://pick_up/meshes/link5.STL; visual mesh filename=package://pick_up/meshes/link5.STL
- link r_in_link: geometry collision mesh filename=package://pick_up/meshes/r_in_link.STL; visual mesh filename=package://pick_up/meshes/r_in_link.STL
- link r_link: geometry collision mesh filename=package://pick_up/meshes/r_link.STL; visual mesh filename=package://pick_up/meshes/r_link.STL
- link r_out_link: geometry collision mesh filename=package://pick_up/meshes/r_out_link.STL; visual mesh filename=package://pick_up/meshes/r_out_link.STL
